File: kicad/ckc-mx.kicad_pcb (KiCad board)
At the start: 2 copper layers, 20 x 22 mm, 7 parts, among them J1 Conn_01x05_Male, SW1 SW_Push

Commit message: updated project
Parts:
- moved J1 0.65 mm to (144.5, 69.8)
Routing:
- net Net-(J1-Pad3): track 4.04 -> 4.69 mm
- net Net-(J1-Pad4): track 3.79 -> 4.44 mm
