File: kicad/ckc-mx.kicad_sch (KiCad schematic)
At the start: 7 parts, among them J1 Conn_01x05_Male, SW1 SW_Push

Commit message: updated project
Other:
- moved on the sheet: R1, R2, R3
Changed lines of the file:
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@@
     (stroke (width 0) (type default) (color 0 0 0 0))
   )
-  (wire (pts (xy 90.17 93.98) (xy 102.87 93.98))
+  (wire (pts (xy 90.17 93.98) (xy 93.98 93.98))
     (stroke (width 0) (type default) (color 0 0 0 0))
   )
@@
     (stroke (width 0) (type default) (color 0 0 0 0))
   )
-  (wire (pts (xy 83.82 83.82) (xy 102.87 83.82))
+  (wire (pts (xy 83.82 83.82) (xy 93.98 83.82))
     (stroke (width 0) (type default) (color 0 0 0 0))
   )
@@
     (stroke (width 0) (type default) (color 0 0 0 0))
   )
-  (wire (pts (xy 102.87 88.9) (xy 91.44 88.9))
+  (wire (pts (xy 93.98 88.9) (xy 91.44 88.9))
     (stroke (width 0) (type default) (color 0 0 0 0))
   )
@@
     (effects (font (size 1.27 1.27)) (justify left bottom))
   )
-  (global_label "d" (shape input) (at 107.95 93.98 0) (fields_autoplaced)
+  (global_label "d" (shape input) (at 99.06 93.98 0) (fields_autoplaced)
     (effects (font (size 1.27 1.27)) (justify left))
-    (property "Intersheet References" "${INTERSHEET_REFS}" (id 0) (at 111.5121 93.9006 0)
+    (property "Intersheet References" "${INTERSHEET_REFS}" (id 0) (at 102.6221 93.9006 0)
       (effects (font (size 1.27 1.27)) (justify left) hide)
     )
@@
     )
   )
-  (global_label "s" (shape input) (at 107.95 83.82 0) (fields_autoplaced)
+  (global_label "s" (shape input) (at 99.06 83.82 0) (fields_autoplaced)
     (effects (font (size 1.27 1.27)) (justify left))
-    (property "Intersheet References" "${INTERSHEET_REFS}" (id 0) (at 111.3912 83.7406 0)
+    (property "Intersheet References" "${INTERSHEET_REFS}" (id 0) (at 102.5012 83.7406 0)
       (effects (font (size 1.27 1.27)) (justify left) hide)
     )
@@
     )
   )
-  (global_label "a" (shape input) (at 107.95 88.9 0) (fields_autoplaced)
+  (global_label "a" (shape input) (at 99.06 88.9 0) (fields_autoplaced)
     (effects (font (size 1.27 1.27)) (justify left))
-    (property "Intersheet References" "${INTERSHEET_REFS}" (id 0) (at 111.5121 88.8206 0)
+    (property "Intersheet References" "${INTERSHEET_REFS}" (id 0) (at 102.6221 88.8206 0)
       (effects (font (size 1.27 1.27)) (justify left) hide)
     )
@@
     (pin "1")
   )
-  (symbol (lib_id "Device:R_Small") (at 105.41 93.98 90) (unit 1)
-    (in_bom yes) (on_board yes)
-    (property "Reference" "R3" (id 0) (at 102.87 91.44 90))
-    (property "Value" "R_Small" (id 1) (at 110.49 91.44 90))
-    (property "Footprint" "Resistor_SMD:R_0805_2012Metric_Pad1.20x1.40mm_HandSolder" (id 2) (at 105.41 93.98 0)
-      (effects (font (size 1.27 1.27)) hide)
-    )
-    (property "Datasheet" "~" (id 3) (at 105.41 93.98 0)
-      (effects (font (size 1.27 1.27)) hide)
-    )
-    (pin "1")
-    (pin "2")
-  )
-  (symbol (lib_id "Device:R_Small") (at 105.41 83.82 90) (unit 1)
-    (in_bom yes) (on_board yes)
-    (property "Reference" "R1" (id 0) (at 102.87 81.28 90))
-    (property "Value" "R_Small" (id 1) (at 110.49 81.28 90))
-    (property "Footprint" "Resistor_SMD:R_0805_2012Metric_Pad1.20x1.40mm_HandSolder" (id 2) (at 105.41 83.82 0)
-      (effects (font (size 1.27 1.27)) hide)
-    )
-    (property "Datasheet" "~" (id 3) (at 105.41 83.82 0)
+  (symbol (lib_id "Device:R_Small") (at 96.52 93.98 90) (unit 1)
+    (in_bom yes) (on_board yes)
+    (property "Reference" "R3" (id 0) (at 93.98 91.44 90))
+    (property "Value" "R_Small" (id 1) (at 101.6 91.44 90))
+    (property "Footprint" "Resistor_SMD:R_0805_2012Metric_Pad1.20x1.40mm_HandSolder" (id 2) (at 96.52 93.98 0)
+      (effects (font (size 1.27 1.27)) hide)
+    )
+    (property "Datasheet" "~" (id 3) (at 96.52 93.98 0)
+      (effects (font (size 1.27 1.27)) hide)
+    )
+    (pin "1")
+    (pin "2")
+  )
+  (symbol (lib_id "Device:R_Small") (at 96.52 83.82 90) (unit 1)
+    (in_bom yes) (on_board yes)
+    (property "Reference" "R1" (id 0) (at 93.98 81.28 90))
+    (property "Value" "R_Small" (id 1) (at 101.6 81.28 90))
+    (property "Footprint" "Resistor_SMD:R_0805_2012Metric_Pad1.20x1.40mm_HandSolder" (id 2) (at 96.52 83.82 0)
+      (effects (font (size 1.27 1.27)) hide)
+    )
+    (property "Datasheet" "~" (id 3) (at 96.52 83.82 0)
       (effects (font (size 1.27 1.27)) hide)
     )
@@
     (pin "4")
   )
-  (symbol (lib_id "Device:R_Small") (at 105.41 88.9 90) (unit 1)
-    (in_bom yes) (on_board yes)
-    (property "Reference" "R2" (id 0) (at 102.87 86.36 90))
-    (property "Value" "R_Small" (id 1) (at 110.49 86.36 90))
-    (property "Footprint" "Resistor_SMD:R_0805_2012Metric_Pad1.20x1.40mm_HandSolder" (id 2) (at 105.41 88.9 0)
-      (effects (font (size 1.27 1.27)) hide)
-    )
-    (property "Datasheet" "~" (id 3) (at 105.41 88.9 0)
-      (effects (font (size 1.27 1.27)) hide)
-    )
+  (symbol (lib_id "Device:R_Small") (at 96.52 88.9 90) (unit 1)
+    (in_bom yes) (on_board yes)
+    (property "Reference" "R2" (id 0) (at 93.98 86.36 90))
+    (property "Value" "R_Small" (id 1) (at 101.6 86.36 90))
+    (property "Footprint" "Resistor_SMD:R_0805_2012Metric_Pad1.20x1.40mm_HandSolder" (id 2) (at 96.52 88.9 0)
+      (effects (font (size 1.27 1.27)) hide)
+    )
+    (property "Datasheet" "~" (id 3) (at 96.52 88.9 0)
+      (effects (font (size 1.27 1.27)) hide)
+    )
